File: hardware-basic/chaos_papagali.kicad_pcb (KiCad board)
At the start: 2 copper layers, 49.4 x 43.7 mm, 41 parts, among them J1 Conn_01x06, J2 USB_B_Micro, J3 BAT, M1 Motor_DC, Q1 BC847, SW1 SW_Push, SW3 SW_DIP_x04, U1 ATmega328P-M, U2 TP4056, U4 FS8205A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

Commit message: First full project commit
Changed lines of the file:
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@@
 		(tags "resistor handsolder")
 		(property "Reference" "R9"
-			(at -2.7705 0.127 -90)
+			(at -2.6435 0 -90)
 			(layer "F.SilkS")
 			(effects
@@
 		(tags "resistor handsolder")
 		(property "Reference" "R10"
-			(at 3.0715 0 90)
+			(at 2.3095 -1.27 90)
 			(layer "F.SilkS")
 			(effects
@@
 		(tags "SOD-123")
 		(property "Reference" "D4"
-			(at 0.127 1.651 180)
+			(at -3.428 -0.381 180)
 			(layer "F.SilkS")
 			(effects
@@
 		)
 		(fp_text user "${REFERENCE}"
-			(at 0.127 1.651 180)
+			(at -3.428 -0.381 180)
 			(layer "F.Fab")
 			(effects
@@
 		(tags "Through hole pin header THT 1x02 2.54mm single row")
 		(property "Reference" "SW1"
-			(at 0 -2.54 180)
+			(at -1.778 -2.54 180)
 			(layer "F.SilkS")
 			(effects
@@
 		(tags "capacitor handsolder")
 		(property "Reference" "C10"
-			(at 0 -1.43 180)
+			(at 2.5665 -0.254 -90)
 			(layer "F.SilkS")
 			(effects
@@
 		(tags "resistor handsolder")
 		(property "Reference" "R2"
-			(at 2.6445 -0.635 0)
+			(at 2.2635 -0.889 0)
 			(layer "F.SilkS")
 			(effects
@@
 		(tags "DIP Switch SPST Slide 7.62mm 300mil")
 		(property "Reference" "SW3"
-			(at -2.032 8.636 90)
+			(at -2.032 3.302 90)
 			(layer "F.SilkS")
 			(effects
@@
 		)
 		(fp_text user "${REFERENCE}"
-			(at -2.032 8.636 90)
+			(at -1.905 3.429 90)
 			(layer "F.Fab")
 			(effects
@@
 		(tags "Through hole pin header THT 1x02 2.54mm single row")
 		(property "Reference" "J3"
-			(at 2.54 4.138 180)
+			(at 2.54 2.032 180)
 			(layer "F.SilkS")
 			(effects
